Commit message: Add impedance-on to marengo-pi; bump right bench URDF mass slightly.
Keep gravity-on as the primary light backdrive path; model mass 82 g (~10% over measured) adds a little support when lifted without changing arm-down feel.

File: assets/urdf/shoulder_pitch_right_bare.urdf (robot description, URDF)
Before this commit: robot shoulder_pitch_right_bare, 2 links, 1 joints
Links:
- link right_upper_arm_stub: mass 0.075 -> 0.082

Commit message: Tune right bench gravity model to 83g and shorten default backdrive to 30s.
Slightly stronger URDF mass for lift support; MCP pi_marengo_pi_script default timeout matches shorter bench sessions.

File: assets/urdf/shoulder_pitch_right_bare.urdf (robot description, URDF)
Before this commit: robot shoulder_pitch_right_bare, 2 links, 1 joints
Links:
- link right_upper_arm_stub: mass 0.082 -> 0.083

Commit message: Add hold-at slew ramp and lock in right shoulder bench tuning.
Ramp position setpoints with configurable slew, max_lead, and trim so hold-at moves feel smooth on hardware; record validated kp=12, 15 rad/s slew, and horizontal limits for the bare right-shoulder profile.

File: assets/urdf/shoulder_pitch_right_bare.urdf (robot description, URDF)
Before this commit: robot shoulder_pitch_right_bare, 2 links, 1 joints
Joints:
- joint right_shoulder_pitch: limit lower=-1.2 upper=1.2 effort=10 velocity=2.0 -> lower=-1.2 upper=1.65 effort=10 velocity=2.0
