Commit message: Mirror shoulder pitch bench tuning to left.

File: assets/urdf/shoulder_pitch_dual.urdf (robot description, URDF)
Before this commit: robot shoulder_pitch_dual, 3 links, 2 joints
Joints:
- joint left_shoulder_pitch: limit lower=-1.2 upper=1.2 effort=10 velocity=2.0 -> lower=-1.2 upper=1.65 effort=10 velocity=2.0
- joint right_shoulder_pitch: limit lower=-1.2 upper=1.2 effort=10 velocity=2.0 -> lower=-1.2 upper=1.65 effort=10 velocity=2.0
