Commit message: feat(bench): weighted gravity sign test prep (M4)
Align shoulder_pitch_weighted.urdf with bare bench geometry, fix pi_bench_harness
to select the weighted config profile, add mass-update script and runbook for
the queued right-side sign validation before repeating left gravity-on.

Co-authored-by: Joey Lamping <jaylamping@users.noreply.github.com>

File: assets/urdf/shoulder_pitch_weighted.urdf (robot description, URDF)
Before this commit: robot shoulder_pitch_weighted, 3 links, 2 joints
Links:
- link base_link: mass 5.0 -> 0.001
- link left_upper_arm_stub: mass 1.5 -> 0.083
- link right_upper_arm_stub: mass 2.3 -> 0.583
Joints:
- joint left_shoulder_pitch: origin xyz=0 0.12 0.35 rpy=0 0 0 -> xyz=0 0 0 rpy=0 0 0
- joint right_shoulder_pitch: origin xyz=0 -0.12 0.35 rpy=0 0 0 -> xyz=0 0 0 rpy=0 0 0

Commit message: fix(mcp): Pi staging install and bench config sync
Deploy uses passwordless sudo install from ~/marengo; add
pi_install_staging and scp fallback on Windows. Set weighted URDF
to 0.7 kg with 18 in COM for right fixture.

File: assets/urdf/shoulder_pitch_weighted.urdf (robot description, URDF)
Before this commit: robot shoulder_pitch_weighted, 3 links, 2 joints
Links:
- link right_upper_arm_stub: mass 0.583 -> 0.7
