Commit message: Set shoulder pitch limits and right sign convention.

File: assets/urdf/arm_4dof.urdf (robot description, URDF)
Before this commit: robot arm_4dof, 5 links, 4 joints
Joints:
- joint shoulder_pitch: limit lower=-1.2 upper=1.2 effort=60 velocity=3.0 -> lower=-0.9 upper=3.17 effort=60 velocity=3.0

File: assets/urdf/shoulder_pitch_dual.urdf (robot description, URDF)
Before this commit: robot shoulder_pitch_dual, 3 links, 2 joints
Joints:
- joint left_shoulder_pitch: limit lower=-1.2 upper=1.65 effort=10 velocity=2.0 -> lower=-0.9 upper=3.17 effort=10 velocity=2.0
- joint right_shoulder_pitch: limit lower=-1.2 upper=1.65 effort=10 velocity=2.0 -> lower=-0.9 upper=3.17 effort=10 velocity=2.0

File: assets/urdf/shoulder_pitch_left_bare.urdf (robot description, URDF)
Before this commit: robot shoulder_pitch_left_bare, 2 links, 1 joints
Joints:
- joint left_shoulder_pitch: limit lower=-1.2 upper=1.65 effort=10 velocity=2.0 -> lower=-0.9 upper=3.17 effort=10 velocity=2.0

File: assets/urdf/shoulder_pitch_right_bare.urdf (robot description, URDF)
Before this commit: robot shoulder_pitch_right_bare, 2 links, 1 joints
Joints:
- joint right_shoulder_pitch: limit lower=-1.2 upper=1.65 effort=10 velocity=2.0 -> lower=-0.9 upper=3.17 effort=10 velocity=2.0

File: assets/urdf/shoulder_pitch_weighted.urdf (robot description, URDF)
Before this commit: robot shoulder_pitch_weighted, 3 links, 2 joints
Joints:
- joint left_shoulder_pitch: limit lower=-1.2 upper=1.2 effort=10 velocity=2.0 -> lower=-0.9 upper=3.17 effort=10 velocity=2.0
- joint right_shoulder_pitch: limit lower=-1.2 upper=1.2 effort=10 velocity=2.0 -> lower=-0.9 upper=3.17 effort=10 velocity=2.0

Commit message: fix(cad): align torso shoulder pitch naming across CAD and SSOT
Rename torso RS03 instances and pitch mount brackets; update kinematics,
arm_4dof URDF chain, and bring-up configs to pitch-on-torso layout.

File: assets/urdf/arm_4dof.urdf (robot description, URDF)
Before this commit: robot arm_4dof, 5 links, 4 joints
Joints:
- joint shoulder_pitch: origin xyz=0.05 0 0 rpy=0 1.57 0 -> xyz=0 0 0.1 rpy=0 0 0; parent shoulder_roll_link -> base_link
- joint shoulder_roll: origin xyz=0 0 0.1 rpy=0 0 0 -> xyz=0.05 0 0 rpy=0 1.57 0; parent base_link -> shoulder_pitch_link
- joint upper_arm_yaw: parent shoulder_pitch_link -> shoulder_roll_link
