Commit message: feat(consul): render URDF primitive visuals in R3F preview
Parse <visual> boxes, cylinders, and spheres from URDF links and render
them in the Consul R3F preview instead of placeholder boxes. Add primitive
visual geometry to shoulder_pitch_right_only.urdf so the shoulder pitch
axis and arm stub orientation are visible for bench verification.

File: assets/urdf/shoulder_pitch_right_only.urdf (robot description, URDF)
Before this commit: robot marengo_shoulder_pitch_right_only, 2 links, 1 joints
Links:
- link base_link: geometry visual cylinder length=0.10 radius=0.04
- link right_upper_arm_stub: geometry visual cylinder length=0.4 radius=0.03

Commit message: feat(bench): model 700g loaded arm in right-only shoulder pitch URDF

File: assets/urdf/shoulder_pitch_right_only.urdf (robot description, URDF)
Before this commit: robot marengo_shoulder_pitch_right_only, 2 links, 1 joints
Links:
- link right_upper_arm_stub: mass 0.083 -> 0.7
