Commit message: feat(bench): roll 2-DOF harness, ki tuning, and suite docs
Add roll_attached/arm_2dof_smoke harness paths with staged return-home,
conservative roll velocity caps, and pitch-proven impedance on arm_2dof_right.
Document roll and 2-DOF smoke protocols; wire explicit ki in config schema.

File: assets/urdf/arm_2dof_right.urdf (robot description, URDF)
Before this commit: robot marengo_arm_2dof_right, 4 links, 3 joints
Joints:
- joint right_shoulder_roll: limit lower=-1.57 upper=1.57 effort=60 velocity=2.0 -> lower=0.0 upper=3.14159 effort=60 velocity=2.0
