Commit message: feat(berthier,consul): native cosine Wave compound test
Drive continuous roll from Berthier PositionWave with analytical velocity,
fix home clamp near hard_lower, and capture Consul product context.

File: assets/urdf/arm_2dof_right.urdf (robot description, URDF)
Before this commit: robot marengo_arm_2dof_right, 4 links, 3 joints
Joints:
- joint right_shoulder_pitch: limit lower=-0.9 upper=3.17 effort=60 velocity=2.0 -> lower=-0.9 upper=3.25 effort=60 velocity=2.0
- joint right_shoulder_roll: limit lower=0.0 upper=3.14159 effort=60 velocity=2.0 -> lower=-0.05 upper=3.14159 effort=60 velocity=2.0
