Commit message: feat(bench): add right upper-arm yaw RS02 and rename to arm_3dof_right
Extend the right-arm bringup with device_id 3 (right_upper_arm_yaw) and
make arm_3dof_right the default bench profile across config, Consul, and MCP.

File: assets/urdf/arm_3dof_right.urdf (robot description, URDF)
Before this commit: robot marengo_arm_2dof_right, 4 links, 3 joints
Links:
- removed link right_upper_arm_stub
- added link right_upper_arm_link, mass 0.7; visual cylinder length=0.4 radius=0.03
Joints:
- removed joint right_upper_arm_fixed
- added joint right_upper_arm_yaw: type revolute, parent right_shoulder_roll_link, child right_upper_arm_link, origin xyz=0.08 0 0 rpy=0 0 0, axis 0 0 1, limit lower=-1.57 upper=1.57 effort=17 velocity=2.0
