Commit message: fix(bench): allow slight negative elbow lower limit at zero
Encoder noise near mechanical zero was ~-0.4 mrad, which tripped Davout
keepalive hard limits when URDF/motors lower was exactly 0 and dropped
Enable back to Disabled.

File: assets/urdf/arm_4dof_right.urdf (robot description, URDF)
Before this commit: robot marengo_arm_4dof_right, 5 links, 4 joints
Joints:
- joint right_elbow_pitch: limit lower=0.0 upper=1.2 effort=17 velocity=2.0 -> lower=-0.05 upper=1.2 effort=17 velocity=2.0

Commit message: feat(limits): expand URDF on Set Limits and wait for Durable persist
Apply Limits now widens hard envelopes everywhere (motors, control soft inset,
expand-only URDF) with a single atomic write path, Durable-gated local git sync,
and clearer Enable hard-limit feedback when URDF still clamps.

File: assets/urdf/arm_4dof_right.urdf (robot description, URDF)
Before this commit: robot marengo_arm_4dof_right, 5 links, 4 joints
Joints:
- joint right_elbow_pitch: limit lower=-0.05 upper=1.2 effort=17 velocity=2.0 -> lower=-0.50 upper=1.2 effort=17 velocity=2.0

Commit message: fix(bench): weigh forearm mass and unlock Wave after E6
Elevated GravityComp runaway was driven by a 0.35 kg provisional forearm;
bench weigh (~75 g) fixes elbow τ_g. Record E6 sign PASS and enable live Wave.

File: assets/urdf/arm_4dof_right.urdf (robot description, URDF)
Before this commit: robot marengo_arm_4dof_right, 5 links, 4 joints
Links:
- link right_forearm_link: mass 0.35 -> 0.075
