Commit message: feat(config): master SoT cutover for consul-hardware-sot phase 1
Collapse arm_4dof_right bench YAML into root config/, promote live
marengo.urdf from the right 4-DOF slice, archive legacy URDFs with
manifests, and retire bringup profile runtime reads in marengo-config.

- Default MARENGO_CONFIG_DIR to /opt/marengo/config when present
- Retarget profile_txn/urdf_expand to master paths; bringup_compat stubs
- Update ADR 0012 disk paths; align MJCF + kinematics fixtures

Co-authored-by: Joey Lamping <jaylamping@users.noreply.github.com>

File: assets/urdf/marengo.urdf (robot description, URDF)
Before this commit: robot marengo, 3 links, 2 joints
Links:
- removed link link1
- removed link link2
- added link right_forearm_link, mass 0.35; visual cylinder length=0.2 radius=0.025
- added link right_shoulder_pitch_link, mass 0.3
- added link right_shoulder_roll_link, mass 0.3
- added link right_upper_arm_link, mass 0.55; visual cylinder length=0.24 radius=0.03
- link base_link: mass 1.0 -> 0.001; geometry visual cylinder length=0.10 radius=0.04
Joints:
- removed joint joint1
- removed joint joint2
- added joint right_elbow_pitch: type revolute, parent right_upper_arm_link, child right_forearm_link, origin xyz=0 0 -0.24 rpy=0 0 0, axis 0 1 0, limit lower=-0.50 upper=1.2 effort=17 velocity=2.0
- added joint right_shoulder_pitch: type revolute, parent base_link, child right_shoulder_pitch_link, origin xyz=0 0 0 rpy=0 0 0, axis 0 1 0, limit lower=-0.9 upper=3.25 effort=60 velocity=2.0
- added joint right_shoulder_roll: type revolute, parent right_shoulder_pitch_link, child right_shoulder_roll_link, origin xyz=0.05 0 0 rpy=0 0 0, axis 1 0 0, limit lower=-0.05 upper=3.14159 effort=60 velocity=2.0
- added joint right_upper_arm_yaw: type revolute, parent right_shoulder_roll_link, child right_upper_arm_link, origin xyz=0.08 0 0 rpy=0 0 0, axis 0 0 1, limit lower=-1.57 upper=1.57 effort=17 velocity=2.0

Commit message: feat(config): add right_lower_arm_yaw as CAN id 5 (5-DOF bench)
Promote master SoT from 4-DOF to 5-DOF: motors/robot/homing/control,
provisional URDF hand link, and docs. RS00 on can0 device_id 5.

Co-authored-by: Joey Lamping <jaylamping@users.noreply.github.com>

File: assets/urdf/marengo.urdf (robot description, URDF)
Before this commit: robot marengo_arm_4dof_right, 5 links, 4 joints
Links:
- added link right_hand_link, mass 0.12; visual cylinder length=0.06 radius=0.02
Joints:
- added joint right_lower_arm_yaw: type revolute, parent right_forearm_link, child right_hand_link, origin xyz=0 0 -0.20 rpy=0 0 0, axis 0 1 0, limit lower=-1.6 upper=1.6 effort=17 velocity=2.0

Commit message: Save cancelled session checkpoint and preserved arm configuration edits

File: assets/urdf/marengo.urdf (robot description, URDF)
Before this commit: robot marengo_arm_5dof_right, 6 links, 5 joints
Joints:
- joint right_lower_arm_yaw: limit lower=-1.6 upper=1.6 effort=17 velocity=2.0 -> lower=-1.6 upper=1.6 effort=14 velocity=2.0
