Commit message: fix(urdf): right-arm joint origins and inertials from CAD
Replace the placeholder right-arm geometry with values read from
cad/assemblies/marengo_arm_right_asm through the SolidWorks MCP:

- Joint origins from the actuator mates: roll axis crosses the pitch axis
  73.5 mm outboard of the pitch output face, upper-arm yaw 1.15 mm off it,
  elbow 230.4 mm below, RS00 output face 99.7 mm below the elbow (was
  0.05/0.08 m forward offsets that put -1.6 Nm on pitch at rest).
- Link mass/COM/inertia: RobStride datasheet masses with CAD COMs, PLA
  parts estimated from CAD volume and area at 20 % infill; hidden
  actuator copies embedded in three part files are excluded.
- Hard limits copied from the Pi's taught URDF (ADR 0017); soft limits and
  axes unchanged. Visual cylinders follow the new spacing.

Predicted tau_g at rest: pitch +0.034, roll -0.026, elbow -0.003 Nm (gate
0.20); pitch tau_g rises to +1.34 Nm at 0.48 rad. Derivation, assumptions
and open items (lower-arm yaw axis, the 2026-08-12 reference) are in
docs/commissioning/right-arm-urdf-from-cad-2026-10-03.md.

Co-Authored-By: Claude Opus 5.5 <noreply@anthropic.com>

File: assets/urdf/marengo.urdf (robot description, URDF)
Before this commit: robot marengo_arm_5dof_right, 6 links, 5 joints
Links:
- link right_forearm_link: mass 0.35 -> 0.3910; geometry visual cylinder length=0.1 radius=0.025
- link right_hand_link: mass 0.12 -> 0.0822; geometry visual cylinder length=0.12 radius=0.02
- link right_shoulder_pitch_link: mass 0.3 -> 1.0101
- link right_shoulder_roll_link: mass 0.3 -> 0.4925
- link right_upper_arm_link: mass 0.55 -> 0.5075; geometry visual cylinder length=0.23 radius=0.03
Joints:
- joint right_elbow_pitch: limit lower=-0.50 upper=1.2 effort=17 velocity=2.0 -> lower=-1.63191 upper=1.60728 effort=17 velocity=2.0; origin xyz=0 0 -0.24 rpy=0 0 0 -> xyz=0 0 -0.23036 rpy=0 0 0
- joint right_lower_arm_yaw: limit lower=-1.6 upper=1.6 effort=17 velocity=2.0 -> lower=-3.24409 upper=3.24409 effort=17 velocity=2.0; origin xyz=0 0 -0.20 rpy=0 0 0 -> xyz=0.00013 0.00006 -0.09968 rpy=0 0 0
- joint right_shoulder_pitch: limit lower=-0.9 upper=3.25 effort=60 velocity=2.0 -> lower=-1.43134 upper=3.25 effort=60 velocity=2.0
- joint right_shoulder_roll: limit lower=-0.05 upper=3.14159 effort=60 velocity=2.0 -> lower=-0.099415 upper=3.22308 effort=60 velocity=2.0; origin xyz=0.05 0 0 rpy=0 0 0 -> xyz=0 0.07349 0 rpy=0 0 0
- joint right_upper_arm_yaw: origin xyz=0.08 0 0 rpy=0 0 0 -> xyz=0.00115 -0.00001 0 rpy=0 0 0
